File: adapter/adapter.kicad_sch (KiCad schematic)
At the start: 18 parts, among them J1 Conn_01x03_Female, J2 Conn_01x06_Female, SW1 RotaryEncoder_Switch

Commit message: Update adapter.kicad_sch
Parts:
- removed D?: SK6812MINI, Library:YS-SK6812MINI-E, symbol LED:SK6812MINI
- gave numbers to parts that had none: 6
Changed lines of the file:
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@@
   (symbol (lib_id "LED:SK6812MINI") (at 229.87 95.25 0) (unit 1)
     (in_bom yes) (on_board yes)
-    (property "Reference" "D?" (id 0) (at 238.76 93.98 0)
+    (property "Reference" "D12" (id 0) (at 238.76 93.98 0)
       (effects (font (size 1.27 1.27)) (justify left))
     )
@@
   (symbol (lib_id "LED:SK6812MINI") (at 173.99 119.38 0) (unit 1)
     (in_bom yes) (on_board yes)
-    (property "Reference" "D?" (id 0) (at 182.88 118.11 0)
+    (property "Reference" "D8" (id 0) (at 182.88 118.11 0)
       (effects (font (size 1.27 1.27)) (justify left))
     )
@@
   (symbol (lib_id "LED:SK6812MINI") (at 220.98 118.11 0) (unit 1)
     (in_bom yes) (on_board yes)
-    (property "Reference" "D?" (id 0) (at 229.87 116.84 0)
+    (property "Reference" "D11" (id 0) (at 229.87 116.84 0)
       (effects (font (size 1.27 1.27)) (justify left))
     )
@@
   (symbol (lib_id "LED:SK6812MINI") (at 203.2 118.11 0) (unit 1)
     (in_bom yes) (on_board yes)
-    (property "Reference" "D?" (id 0) (at 212.09 116.84 0)
+    (property "Reference" "D9" (id 0) (at 212.09 116.84 0)
       (effects (font (size 1.27 1.27)) (justify left))
     )
@@
   (symbol (lib_id "LED:SK6812MINI") (at 156.21 119.38 0) (unit 1)
     (in_bom yes) (on_board yes)
-    (property "Reference" "D?" (id 0) (at 165.1 118.11 0)
+    (property "Reference" "D7" (id 0) (at 165.1 118.11 0)
       (effects (font (size 1.27 1.27)) (justify left))
     )
@@
     (pin "S2")
   )
-  (symbol (lib_id "LED:SK6812MINI") (at 252.73 123.19 0) (unit 1)
-    (in_bom yes) (on_board yes)
-    (property "Reference" "D?" (id 0) (at 261.62 121.92 0)
-      (effects (font (size 1.27 1.27)) (justify left))
-    )
-    (property "Value" "SK6812MINI" (id 1) (at 261.62 124.46 0)
-      (effects (font (size 1.27 1.27)) (justify left))
-    )
-    (property "Footprint" "Library:YS-SK6812MINI-E" (id 2) (at 254 130.81 0)
-      (effects (font (size 1.27 1.27)) (justify left top) hide)
-    )
-    (property "Datasheet" "https://cdn-shop.adafruit.com/product-files/2686/SK6812MINI_REV.01-1-2.pdf" (id 3) (at 255.27 132.715 0)
-      (effects (font (size 1.27 1.27)) (justify left top) hide)
-    )
-    (pin "1")
-    (pin "2")
-    (pin "3")
-    (pin "4")
-  )
   (symbol (lib_id "Connector:Conn_01x03_Female") (at 39.37 73.66 0) (unit 1)
     (in_bom yes) (on_board yes)
@@
   (symbol (lib_id "LED:SK6812MINI") (at 212.09 95.25 0) (unit 1)
     (in_bom yes) (on_board yes)
-    (property "Reference" "D?" (id 0) (at 220.98 93.98 0)
+    (property "Reference" "D10" (id 0) (at 220.98 93.98 0)
       (effects (font (size 1.27 1.27)) (justify left))
     )
@@
       (reference "D6") (unit 1) (value "SK6812MINI") (footprint "Library:YS-SK6812MINI-E")
     )
+    (path "/cc7bddcd-c8e8-4e37-b9f8-812479985d0d"
+      (reference "D7") (unit 1) (value "SK6812MINI") (footprint "Library:YS-SK6812MINI-E")
+    )
+    (path "/2c01d037-4d82-4530-a305-adce89390391"
+      (reference "D8") (unit 1) (value "SK6812MINI") (footprint "Library:YS-SK6812MINI-E")
+    )
+    (path "/619f1226-0090-432d-9f3b-99c45e391ff3"
+      (reference "D9") (unit 1) (value "SK6812MINI") (footprint "Library:YS-SK6812MINI-E")
+    )
+    (path "/fd6c28ca-f403-4b61-93f7-9bd443c68cc9"
+      (reference "D10") (unit 1) (value "SK6812MINI") (footprint "Library:YS-SK6812MINI-E")
+    )
+    (path "/525ce5ad-fe7e-42fb-9037-c6b7bd02190e"
+      (reference "D11") (unit 1) (value "SK6812MINI") (footprint "Library:YS-SK6812MINI-E")
+    )
     (path "/0984c8a3-e1fc-4d24-8e6e-9c4ba5a77a66"
-      (reference "D?") (unit 1) (value "SK6812MINI") (footprint "Library:YS-SK6812MINI-E")
-    )
-    (path "/2c01d037-4d82-4530-a305-adce89390391"
-      (reference "D?") (unit 1) (value "SK6812MINI") (footprint "Library:YS-SK6812MINI-E")
-    )
-    (path "/525ce5ad-fe7e-42fb-9037-c6b7bd02190e"
-      (reference "D?") (unit 1) (value "SK6812MINI") (footprint "Library:YS-SK6812MINI-E")
-    )
-    (path "/619f1226-0090-432d-9f3b-99c45e391ff3"
-      (reference "D?") (unit 1) (value "SK6812MINI") (footprint "Library:YS-SK6812MINI-E")
-    )
-    (path "/cc7bddcd-c8e8-4e37-b9f8-812479985d0d"
-      (reference "D?") (unit 1) (value "SK6812MINI") (footprint "Library:YS-SK6812MINI-E")
-    )
-    (path "/d9305d58-d25c-4a21-8932-5d0549c8216a"
-      (reference "D?") (unit 1) (value "SK6812MINI") (footprint "Library:YS-SK6812MINI-E")
-    )
-    (path "/fd6c28ca-f403-4b61-93f7-9bd443c68cc9"
-      (reference "D?") (unit 1) (value "SK6812MINI") (footprint "Library:YS-SK6812MINI-E")
+      (reference "D12") (unit 1) (value "SK6812MINI") (footprint "Library:YS-SK6812MINI-E")
     )
     (path "/eb54f150-1815-419c-99e6-8c3c5774df70"
