File: adapter/_autosave-adapter.kicad_sch (KiCad schematic)
At the start: 18 parts, among them J1 Conn_01x03_Female, J2 Conn_01x06_Female, SW1 RotaryEncoder_Switch

Commit message: routing
Connections:
- net ec renamed r1
- net r1: now also SW1.B
- net eda renamed r2
- net r2: now also J2.4 (Pin_4)
- removed net edb: J2.4 (Pin_4), SW1.B
- net er renamed button
Changed lines of the file:
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@@
   )
   (no_connect (at 154.686 117.094))
-  (bus_entry (at 95.504 41.402) (size 2.54 2.54)
-    (stroke (width 0) (type default) (color 0 0 0 0))
-  )
   (wire (pts (xy 162.56 95.25) (xy 165.1 95.25))
     (stroke (width 0) (type default) (color 0 0 0 0))
@@
     )
   )
-  (global_label "er" (shape input) (at 35.56 36.83 180) (fields_autoplaced)
+  (global_label "button" (shape input) (at 35.56 36.83 180) (fields_autoplaced)
     (effects (font (size 1.1938 1.1938)) (justify right))
-    (property "Intersheet References" "${INTERSHEET_REFS}" (id 0) (at 31.3505 36.7554 0)
+    (property "Intersheet References" "${INTERSHEET_REFS}" (id 0) (at 27.428 36.7554 0)
       (effects (font (size 1.1938 1.1938)) (justify right) hide)
     )
@@
     )
   )
-  (global_label "er" (shape input) (at 77.47 35.56 180) (fields_autoplaced)
+  (global_label "button" (shape input) (at 77.47 35.56 180) (fields_autoplaced)
     (effects (font (size 1.1938 1.1938)) (justify right))
-    (property "Intersheet References" "${INTERSHEET_REFS}" (id 0) (at 73.2605 35.4854 0)
+    (property "Intersheet References" "${INTERSHEET_REFS}" (id 0) (at 69.338 35.4854 0)
       (effects (font (size 1.1938 1.1938)) (justify right) hide)
     )
@@
     )
   )
-  (global_label "edb" (shape input) (at 35.56 41.91 180) (fields_autoplaced)
+  (global_label "r2" (shape input) (at 35.56 41.91 180) (fields_autoplaced)
     (effects (font (size 1.1938 1.1938)) (justify right))
-    (property "Intersheet References" "${INTERSHEET_REFS}" (id 0) (at 30.1919 41.9846 0)
+    (property "Intersheet References" "${INTERSHEET_REFS}" (id 0) (at 31.2368 41.8354 0)
       (effects (font (size 1.1938 1.1938)) (justify right) hide)
     )
   )
-  (global_label "eda" (shape input) (at 92.71 40.64 0) (fields_autoplaced)
+  (global_label "r2" (shape input) (at 92.71 40.64 0) (fields_autoplaced)
     (effects (font (size 1.1938 1.1938)) (justify left))
-    (property "Intersheet References" "${INTERSHEET_REFS}" (id 0) (at 98.0781 40.5654 0)
+    (property "Intersheet References" "${INTERSHEET_REFS}" (id 0) (at 97.0332 40.5654 0)
       (effects (font (size 1.1938 1.1938)) (justify left) hide)
     )
   )
-  (global_label "ec" (shape input) (at 35.56 39.37 180) (fields_autoplaced)
+  (global_label "r1" (shape input) (at 35.56 39.37 180) (fields_autoplaced)
     (effects (font (size 1.1938 1.1938)) (justify right))
-    (property "Intersheet References" "${INTERSHEET_REFS}" (id 0) (at 31.0663 39.2954 0)
+    (property "Intersheet References" "${INTERSHEET_REFS}" (id 0) (at 31.2368 39.2954 0)
       (effects (font (size 1.1938 1.1938)) (justify right) hide)
     )
@@
     )
   )
-  (global_label "edb" (shape input) (at 92.71 35.56 0) (fields_autoplaced)
+  (global_label "r1" (shape input) (at 92.71 35.56 0) (fields_autoplaced)
     (effects (font (size 1.1938 1.1938)) (justify left))
-    (property "Intersheet References" "${INTERSHEET_REFS}" (id 0) (at 98.0781 35.4854 0)
+    (property "Intersheet References" "${INTERSHEET_REFS}" (id 0) (at 97.0332 35.4854 0)
       (effects (font (size 1.1938 1.1938)) (justify left) hide)
     )
@@
   (symbol (lib_id "power:GND") (at 75.946 41.402 0) (unit 1)
     (in_bom yes) (on_board yes)
-    (property "Reference" "#PWR?" (id 0) (at 75.946 47.752 0)
+    (property "Reference" "#PWR0105" (id 0) (at 75.946 47.752 0)
       (effects (font (size 1.27 1.27)) hide)
     )
@@
     )
     (path "/f298f139-b4e7-4161-948f-e52265423988"
-      (reference "#PWR?") (unit 1) (value "GND") (footprint "")
+      (reference "#PWR0105") (unit 1) (value "GND") (footprint "")
     )
     (path "/b720e53b-ae72-4295-b3ff-de5411507232"
