File: adapter/adapter.kicad_pcb (KiCad board)
At the start: 2 copper layers, 43.5 x 38.6 mm, 15 parts, among them J1 Conn_01x03_Female, J2 Conn_01x06_Female, SW1 RotaryEncoder_Switch

Commit message: routing
Parts:
- added G*** (x2): LOGO, LOGO, F.Cu at (52.5, 43.6)
- moved D2 1.24 mm to (52.5, 30.2)
- moved D8 1.07 mm to (52.5, 57.3)
- moved D1 0.58 mm to (66.0, 43.6)
- moved D6 0.53 mm to (40.0, 37.1)
- moved D10 0.27 mm to (38.9, 43.6)
Connections:
- net er renamed button
- D10 pad 1: unconnected-(D10-Pad1) -> Net-(D12-Pad3)
- D10 pad 2: unconnected-(D10-Pad2) -> Gnd
- D10 pad 3: unconnected-(D10-Pad3) -> Net-(D10-Pad3)
- D10 pad 4: unconnected-(D10-Pad4) -> Vcc
- D11 pad 2: unconnected-(D11-Pad2) -> Gnd
- D11 pad 3: unconnected-(D11-Pad3) -> Net-(D11-Pad3)
- D11 pad 4: unconnected-(D11-Pad4) -> Vcc
- D12 pad 1: unconnected-(D12-Pad1) -> Net-(D12-Pad1)
- D12 pad 2: unconnected-(D12-Pad2) -> Gnd
- D12 pad 3: unconnected-(D12-Pad3) -> Net-(D12-Pad3)
- D12 pad 4: unconnected-(D12-Pad4) -> Vcc
- D2 pad 1: unconnected-(D2-Pad1) -> Net-(D4-Pad3)
- D2 pad 2: unconnected-(D2-Pad2) -> Gnd
- D2 pad 3: unconnected-(D2-Pad3) -> Net-(D2-Pad3)
- D2 pad 4: unconnected-(D2-Pad4) -> Vcc
- D4 pad 1: unconnected-(D4-Pad1) -> Net-(D4-Pad1)
- D4 pad 2: unconnected-(D4-Pad2) -> Gnd
- D4 pad 3: unconnected-(D4-Pad3) -> Net-(D4-Pad3)
- D4 pad 4: unconnected-(D4-Pad4) -> Vcc
- D5 pad 1: unconnected-(D5-Pad1) -> Net-(D2-Pad3)
- D6 pad 1: unconnected-(D6-Pad1) -> Net-(D10-Pad3)
- D6 pad 2: unconnected-(D6-Pad2) -> Gnd
- D6 pad 3: unconnected-(D6-Pad3) -> Net-(D4-Pad1)
- D6 pad 4: unconnected-(D6-Pad4) -> Vcc
- D7 pad 1: unconnected-(D7-Pad1) -> Net-(D7-Pad1)
- D7 pad 2: unconnected-(D7-Pad2) -> Gnd
- D7 pad 3: unconnected-(D7-Pad3) -> Net-(D12-Pad1)
- D7 pad 4: unconnected-(D7-Pad4) -> Vcc
- D8 pad 1: unconnected-(D8-Pad1) -> Net-(D8-Pad1)
- D8 pad 2: unconnected-(D8-Pad2) -> Gnd
- D8 pad 3: unconnected-(D8-Pad3) -> Net-(D7-Pad1)
- D8 pad 4: unconnected-(D8-Pad4) -> Vcc
- D9 pad 1: unconnected-(D9-Pad1) -> Net-(D11-Pad3)
- D9 pad 2: unconnected-(D9-Pad2) -> Gnd
- D9 pad 3: unconnected-(D9-Pad3) -> Net-(D8-Pad1)
- D9 pad 4: unconnected-(D9-Pad4) -> Vcc
- J2 pad 1: +5V -> Vcc
- J2 pad 3: ec -> r1
- J2 pad 4: edb -> r2
- J2 pad 6: GND -> Gnd
- SW1 pad A: eda -> r2
- SW1 pad B: edb -> r1
- SW1 pad C: GND -> Gnd
- SW1 pad S1: ec -> Gnd
Routing:
- net Vcc: track 0.00 -> 111.3 mm
- net r2: track 0.00 -> 45.0 mm
- net r1: track 0.00 -> 35.0 mm
- net button: track 0.00 -> 20.9 mm
- net Net-(D1-Pad1): track 0.00 -> 18.2 mm
- net Net-(D7-Pad1): track 0.00 -> 17.7 mm
- net Net-(D12-Pad3): track 0.00 -> 17.5 mm
- net Net-(D11-Pad3): track 0.00 -> 17.2 mm
- net Net-(D2-Pad3): track 0.00 -> 16.9 mm
- net Net-(D4-Pad1): track 0.00 -> 16.8 mm
- net Net-(D4-Pad3): track 0.00 -> 16.7 mm
- net Net-(D12-Pad1): track 0.00 -> 16.7 mm
- net Net-(D10-Pad3): track 0.00 -> 16.3 mm
- net Net-(D3-Pad1): track 0.00 -> 16.0 mm
- net Net-(D8-Pad1): track 0.00 -> 15.9 mm
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- added copper zone on B.Cu, net Gnd
- added copper zone on F.Cu, net Gnd
- added copper zone on B.Cu, net Vcc
- removed copper zone on F.Cu, net GND

Commit message: routing, add R C
Parts:
- removed J1: Conn_01x03_Female, Connector_PinHeader_2.54mm:PinHeader_1x03_P2.54mm_Vertical
- added C1: 1u, Capacitor_SMD:C_1206_3216Metric_Pad1.33x1.80mm_HandSolder, F.Cu at (70.0, 38.4)
- added R1: R, Resistor_SMD:R_1206_3216Metric_Pad1.30x1.75mm_HandSolder, F.Cu at (69.5, 48.3)
- turned D1 to 0 degrees
- turned D10 to 180 degrees
- turned D11 to -30 degrees
- turned D12 to -150 degrees
- turned D2 to 90 degrees
- turned D3 to 30 degrees
- turned D4 to 120 degrees
- turned D5 to 60 degrees
- turned D6 to 150 degrees
- turned D7 to -120 degrees
- turned D8 to -90 degrees
- turned D9 to -60 degrees
Connections:
- SW1 pad S1: Gnd -> Vcc
Routing:
- net Vcc: track 111.3 -> 4.69 mm
- net r2: track 45.0 -> 33.4 mm
- net Net-(D1-Pad1): track 18.2 -> 8.12 mm
- net Net-(D11-Pad3): track 17.2 -> 7.35 mm
- net Net-(D1-Pad3): track 0.00 -> 9.48 mm
- net Net-(D7-Pad1): track 17.7 -> 8.75 mm
- net Net-(D10-Pad1): track 17.5 -> 8.62 mm
- net Net-(D2-Pad3): track 16.9 -> 8.27 mm
- net (no net): track 8.39 -> 0.00 mm
- net Gnd: track 15.3 -> 7.11 mm
- net Net-(D4-Pad1): track 16.8 -> 8.78 mm
- net Net-(D10-Pad3): track 16.3 -> 8.34 mm
- net Net-(D12-Pad1): track 16.7 -> 8.91 mm
- net Net-(D2-Pad1): track 16.7 -> 9.12 mm
- net Net-(D3-Pad1): track 16.0 -> 8.73 mm
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- added copper zone on F.Cu, net Vcc
- removed copper zone on B.Cu, net Gnd

Commit message: logo
Parts:
- added G***: LOGO, LOGO, B.Cu at (52.3, 43.9)

Commit message: logos
Other:
- board text added: "BASTARDKB"
- board text added: "REV 1.0"
Changed lines of the file:
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@@
     (effects (font (size 0.8 0.8) (thickness 0.15)))
+  )
+  (gr_text "BASTARDKB" (at 48.4 30.8 90) (layer "F.SilkS")
+    (effects (font (size 0.8 0.8) (thickness 0.12)))
   )
   (gr_text "CS" (at 72 39.810001 45) (layer "F.SilkS")
@@
     (effects (font (size 0.8 0.8) (thickness 0.15)))
   )
+  (gr_text "REV 1.0" (at 49.7 31.809523 90) (layer "F.SilkS")
+    (effects (font (size 0.8 0.8) (thickness 0.12)))
+  )
   (segment (start 70.3425 37.18) (end 70 36.8375) (width 1) (layer "F.Cu") (net 1))

Commit message: license
Parts:
- renumbered C1 to C, R1 to R
Other:
- board text added: "1uF"
- board text added: "330"
- board text added: "BTN"
- board text added: "CHARYBDIS ROTARY ENCODER"
- board text added: "R1"
- board text added: "R2"
- board text added: "RGB"
- board text added: "VCC"
- board text removed: "5V"
- board text removed: "CS"
- board text removed: "MISO"
- board text removed: "MOSI"
- board text removed: "SCLK"
Changed lines of the file:
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@@
         (xy -0.05902 -4.158125)
         (xy 0.011604 -4.158163)
-      ) (layer "F.Cu") (width 0) (fill solid))
+      ) (layer "F.SilkS") (width 0) (fill solid))
   )
   (footprint "Library:YS-SK6812MINI-E" (layer "F.Cu")
@@
     (property "Sheetname" "")
     (attr smd)
-    (fp_text reference "C1" (at 0 0 90) (layer "F.SilkS")
-      (effects (font (size 1 1) (thickness 0.15)))
+    (fp_text reference "C" (at 0 0 90) (layer "F.SilkS")
+      (effects (font (size 0.75 0.75) (thickness 0.1)))
     )
     (fp_text value "1u" (at 0 1.85 90) (layer "F.Fab")
@@
       (effects (font (size 0.8 0.8) (thickness 0.12)))
     )
-    (fp_line (start -0.711252 -0.91) (end 0.711252 -0.91) (layer "F.SilkS") (width 0.12))
-    (fp_line (start -0.711252 0.91) (end 0.711252 0.91) (layer "F.SilkS") (width 0.12))
     (fp_line (start -2.48 -1.15) (end 2.48 -1.15) (layer "F.CrtYd") (width 0.05))
     (fp_line (start 2.48 1.15) (end -2.48 1.15) (layer "F.CrtYd") (width 0.05))
@@
     (fp_line (start 1.6 -0.8) (end 1.6 0.8) (layer "F.Fab") (width 0.1))
     (fp_line (start -1.6 -0.8) (end 1.6 -0.8) (layer "F.Fab") (width 0.1))
-    (pad "1" smd roundrect locked (at -1.5625 0 270) (size 1.325 1.8) (layers "F.Cu" "F.Paste" "F.Mask") (roundrect_rratio 0.188679)
+    (pad "1" smd roundrect (at -1.5625 0 270) (size 1.325 1.8) (layers "F.Cu" "F.Paste" "F.Mask") (roundrect_rratio 0.188679)
       (net 1 "Vcc") (pintype "passive"))
-    (pad "2" smd roundrect locked (at 1.5625 0 270) (size 1.325 1.8) (layers "F.Cu" "F.Paste" "F.Mask") (roundrect_rratio 0.188679)
+    (pad "2" smd roundrect (at 1.5625 0 270) (size 1.325 1.8) (layers "F.Cu" "F.Paste" "F.Mask") (roundrect_rratio 0.188679)
       (net 2 "Gnd") (pintype "passive"))
-    (model "${KICAD6_3DMODEL_DIR}/Capacitor_SMD.3dshapes/C_1206_3216Metric.wrl"
+    (model "${KICAD6_3DMODEL_DIR}/Capacitor_SMD.3dshapes/C_1206_3216Metric.wrl" hide
       (offset (xyz 0 0 0))
       (scale (xyz 1 1 1))
@@
     (property "Sheetname" "")
     (attr smd)
-    (fp_text reference "R1" (at 0 0.1 90) (layer "F.SilkS")
-      (effects (font (size 1 1) (thickness 0.15)))
+    (fp_text reference "R" (at 0 0.1 90) (layer "F.SilkS")
+      (effects (font (size 0.75 0.75) (thickness 0.1)))
     )
     (fp_text value "R" (at 0 1.82 90) (layer "F.Fab")
@@
       (effects (font (size 0.8 0.8) (thickness 0.12)))
     )
-    (fp_line (start -0.727064 0.91) (end 0.727064 0.91) (layer "F.SilkS") (width 0.12))
-    (fp_line (start -0.727064 -0.91) (end 0.727064 -0.91) (layer "F.SilkS") (width 0.12))
     (fp_line (start -2.45 -1.12) (end 2.45 -1.12) (layer "F.CrtYd") (width 0.05))
     (fp_line (start -2.45 1.12) (end -2.45 -1.12) (layer "F.CrtYd") (width 0.05))
@@
     (fp_line (start 1.6 -0.8) (end 1.6 0.8) (layer "F.Fab") (width 0.1))
     (fp_line (start 1.6 0.8) (end -1.6 0.8) (layer "F.Fab") (width 0.1))
-    (pad "1" smd roundrect locked (at -1.55 0 90) (size 1.3 1.75) (layers "F.Cu" "F.Paste" "F.Mask") (roundrect_rratio 0.192308)
+    (pad "1" smd roundrect (at -1.55 0 90) (size 1.3 1.75) (layers "F.Cu" "F.Paste" "F.Mask") (roundrect_rratio 0.192308)
       (net 3 "Net-(D1-Pad3)") (pintype "passive"))
-    (pad "2" smd roundrect locked (at 1.55 0 90) (size 1.3 1.75) (layers "F.Cu" "F.Paste" "F.Mask") (roundrect_rratio 0.192308)
+    (pad "2" smd roundrect (at 1.55 0 90) (size 1.3 1.75) (layers "F.Cu" "F.Paste" "F.Mask") (roundrect_rratio 0.192308)
       (net 6 "rgb") (pintype "passive"))
-    (model "${KICAD6_3DMODEL_DIR}/Resistor_SMD.3dshapes/R_1206_3216Metric.wrl"
+    (model "${KICAD6_3DMODEL_DIR}/Resistor_SMD.3dshapes/R_1206_3216Metric.wrl" hide
       (offset (xyz 0 0 0))
       (scale (xyz 1 1 1))
@@
   (gr_line (start 102.976 17.735) (end 102.976 16.295) (layer "B.CrtYd") (width 0.05))
   (gr_circle (center 52.5 43.6) (end 67 56.85) (layer "F.Fab") (width 0.1) (fill none))
-  (gr_text "MOSI" (at 72.13 42.27 -45) (layer "B.SilkS")
-    (effects (font (size 0.8 0.8) (thickness 0.15)) (justify mirror))
-  )
-  (gr_text "GND" (at 72.13 49.890001 -45) (layer "B.SilkS")
-    (effects (font (size 0.8 0.8) (thickness 0.15)) (justify mirror))
-  )
-  (gr_text "CS" (at 72.13 39.730001 -45) (layer "B.SilkS")
-    (effects (font (size 0.8 0.8) (thickness 0.15)) (justify mirror))
-  )
-  (gr_text "5V" (at 72.13 37.190001 -45) (layer "B.SilkS")
-    (effects (font (size 0.8 0.8) (thickness 0.15)) (justify mirror))
-  )
-  (gr_text "SCLK" (at 72.08 44.81 -45) (layer "B.SilkS")
-    (effects (font (size 0.8 0.8) (thickness 0.15)) (justify mirror))
-  )
-  (gr_text "MISO" (at 72.0546 47.35 -45) (layer "B.SilkS")
-    (effects (font (size 0.8 0.8) (thickness 0.15)) (justify mirror))
-  )
-  (gr_text "SCLK" (at 72.05 44.89 45) (layer "F.SilkS")
-    (effects (font (size 0.8 0.8) (thickness 0.15)))
-  )
-  (gr_text "5V" (at 72 37.270001 45) (layer "F.SilkS")
-    (effects (font (size 0.8 0.8) (thickness 0.15)))
-  )
-  (gr_text "MOSI" (at 72 42.35 45) (layer "F.SilkS")
-    (effects (font (size 0.8 0.8) (thickness 0.15)))
-  )
-  (gr_text "MISO" (at 72.0754 47.43 45) (layer "F.SilkS")
-    (effects (font (size 0.8 0.8) (thickness 0.15)))
-  )
-  (gr_text "BASTARDKB" (at 48.4 30.8 90) (layer "F.SilkS")
-    (effects (font (size 0.8 0.8) (thickness 0.12)))
-  )
-  (gr_text "CS" (at 72 39.810001 45) (layer "F.SilkS")
-    (effects (font (size 0.8 0.8) (thickness 0.15)))
-  )
-  (gr_text "GND" (at 72 49.970001 45) (layer "F.SilkS")
-    (effects (font (size 0.8 0.8) (thickness 0.15)))
-  )
-  (gr_text "REV 1.0" (at 49.7 31.809523 90) (layer "F.SilkS")
-    (effects (font (size 0.8 0.8) (thickness 0.12)))
+  (gr_text "R1" (at 72.6 42.7 45) (layer "F.SilkS")
+    (effects (font (size 0.75 0.75) (thickness 0.1)))
+  )
+  (gr_text "GND" (at 72.309581 50.320001 45) (layer "F.SilkS")
+    (effects (font (size 0.75 0.75) (thickness 0.1)))
+  )
+  (gr_text "BTN" (at 72.372715 40.160001 45) (layer "F.SilkS")
+    (effects (font (size 0.75 0.75) (thickness 0.1)))
+  )
+  (gr_text "BASTARDKB" (at 55 57.3 270) (layer "F.SilkS")
+    (effects (font (size 0.75 0.75) (thickness 0.1)))
+  )
+  (gr_text "330" (at 67.8 48.2 90) (layer "F.SilkS")
+    (effects (font (size 0.75 0.75) (thickness 0.1)))
+  )
+  (gr_text "CHARYBDIS \nROTARY \nENCODER" (at 48.6 26.3 270) (layer "F.SilkS")
+    (effects (font (size 0.75 0.75) (thickness 0.1)) (justify left))
+  )
+  (gr_text "VCC" (at 72.360088 37.620001 45) (layer "F.SilkS")
+    (effects (font (size 0.75 0.75) (thickness 0.1)))
+  )
+  (gr_text "1uF" (at 68.2 38.3 90) (layer "F.SilkS")
+    (effects (font (size 0.75 0.75) (thickness 0.1)))
+  )
+  (gr_text "R2" (at 72.6 45.24 45) (layer "F.SilkS")
+    (effects (font (size 0.75 0.75) (thickness 0.1)))
+  )
+  (gr_text "RGB" (at 72.322208 47.78 45) (layer "F.SilkS")
+    (effects (font (size 0.75 0.75) (thickness 0.1)))
+  )
+  (gr_text "REV 1.0" (at 55 28.6 270) (layer "F.SilkS")
+    (effects (font (size 0.75 0.75) (thickness 0.1)))
   )
   (segment (start 70.3425 37.18) (end 70 36.8375) (width 1) (layer "F.Cu") (net 1))
@@
     )
   )
-  (group "" (id 60bd8311-1652-425b-b4d9-0460ddb21a57)
-    (members
-      0f3a778f-8b61-48da-bc9f-03d466581ce1
-      1b58f4ca-6ef5-48a0-a544-c1e61524b9d2
-      423aa899-df18-4eef-a7fe-cb78efb45f86
-      725e893b-995a-48e5-bd69-5ad21b4afe74
-      d8cf0f21-0e7f-4972-9cfc-5dd7cd4558a4
-      f76b67e4-6fc8-4c99-8f47-e5f4ac236ff6
-    )
-  )

Commit message: silkscreen
Other:
- board text added: "Licensed under CERN-OHL-W v2"
Changed lines of the file:
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@@
   (gr_line (start 102.976 17.735) (end 102.976 16.295) (layer "B.CrtYd") (width 0.05))
   (gr_circle (center 52.5 43.6) (end 67 56.85) (layer "F.Fab") (width 0.1) (fill none))
+  (gr_text "Licensed under\nCERN-OHL-W v2" (at 50.3 51.55 -105) (layer "F.SilkS")
+    (effects (font (size 0.75 0.75) (thickness 0.1)) (justify left))
+  )
   (gr_text "R1" (at 72.6 42.7 45) (layer "F.SilkS")
     (effects (font (size 0.75 0.75) (thickness 0.1)))
@@
     (effects (font (size 0.75 0.75) (thickness 0.1)))
   )
-  (gr_text "BASTARDKB" (at 55 57.3 270) (layer "F.SilkS")
+  (gr_text "BASTARDKB" (at 55.95 56.3 285) (layer "F.SilkS")
     (effects (font (size 0.75 0.75) (thickness 0.1)))
   )
@@
     (effects (font (size 0.75 0.75) (thickness 0.1)))
   )
-  (gr_text "CHARYBDIS \nROTARY \nENCODER" (at 48.6 26.3 270) (layer "F.SilkS")
+  (gr_text "CHARYBDIS \nROTARY \nENCODER" (at 47.3 26.45 285) (layer "F.SilkS")
     (effects (font (size 0.75 0.75) (thickness 0.1)) (justify left))
   )
@@
     (effects (font (size 0.75 0.75) (thickness 0.1)))
   )
-  (gr_text "REV 1.0" (at 55 28.6 270) (layer "F.SilkS")
+  (gr_text "REV 1.0" (at 56.2 30.05 255) (layer "F.SilkS")
     (effects (font (size 0.75 0.75) (thickness 0.1)))
   )
