File: adapter/adapter.kicad_pcb (KiCad board)
At the start: 2 copper layers, 43.5 x 38.6 mm, 26 parts, among them J1 Conn_01x06_Female, J2 Conn_01x01_Female, J5 Conn_01x01_Female, SW1 RotaryEncoder_Switch

Commit message: cleanup for 1.2 release
Other:
- board text added: "REV 1.2"
- board text removed: "REV 1.1.2"
Changed lines of the file:
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@@
       (drillshape 0)
       (scaleselection 1)
-      (outputdirectory "gerbers")
+      (outputdirectory "../../Charybdis-EC11-rev1-2_gerbers/")
     )
   )
@@
     (effects (font (size 0.75 0.75) (thickness 0.1)))
   )
-  (gr_text "REV 1.1.2" (at 56.2 30.05 255) (layer "F.SilkS")
+  (gr_text "REV 1.2" (at 56.2 30.05 255) (layer "F.SilkS")
     (effects (font (size 0.75 0.75) (thickness 0.1)))
   )
